File: Electronics/Controller/Tandem Leveller Controller.kicad_sch (KiCad schematic)
At the start: 4 parts, among them J1 Conn_01x02, U1 TEENSY 4.0

Commit message: Added 4.7uF caps to FT232RL on controller.
Parts:
- J1: LCSC (none) -> C7494857
- R1: value 287 -> 330; LCSC (none) -> C17630
- U1: LCSC (none) -> C2897377
Changed lines of the file:
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@@
   (title_block
     (title "Tandem Leveller Controller")
-    (date "2025-02-22")
+    (date "2025-03-11")
     (rev "V1.0")
     (company "(C) andy@britishideas.com 2025")
@@
       (effects (font (size 1.27 1.27)) hide)
     )
+    (property "LCSC" "C7494857" (at 98.425 43.18 0)
+      (effects (font (size 1.27 1.27)) hide)
+    )
     (pin "1")
     (pin "2")
@@
       (effects (font (size 1.27 1.27)) hide)
     )
+    (property "LCSC" "" (at 195.58 33.655 0)
+      (effects (font (size 1.27 1.27)) hide)
+    )
     (pin "1")
     (pin "2")
@@
     )
     (property "Datasheet" "" (at 83.185 173.355 0)
+      (effects (font (size 1.27 1.27)) hide)
+    )
+    (property "LCSC" "C2897377" (at 83.185 173.355 0)
       (effects (font (size 1.27 1.27)) hide)
     )
@@
       (effects (font (size 1.27 1.27)) (justify left))
     )
-    (property "Value" "287" (at 198.12 44.45 0)
+    (property "Value" "330" (at 198.12 44.45 0)
       (effects (font (size 1.27 1.27)) (justify left))
     )
@@
       (effects (font (size 1.27 1.27)) hide)
     )
+    (property "LCSC" "C17630" (at 195.58 43.18 0)
+      (effects (font (size 1.27 1.27)) hide)
+    )
