File: Electronics/Controller/Power.kicad_sch (KiCad schematic)
At the start: 29 parts, among them J11 TRACTOR BATTERY, J12 PWR SWITCH, J13 VALVE POWER, J14 TABLET 1 PWR, J15 TABLET 2 PWR, U7 LM2596S-5, U8 LM2587S-ADJ/NOPB, U9 LM2587S-ADJ/NOPB

Commit message: Added 4.7uF caps to FT232RL on controller.
Parts:
- C10, C9: LCSC (none) -> C1984785
- C3: LCSC (none) -> C50456
- C4: LCSC (none) -> C3340
- C5, C6: LCSC (none) -> C340733
- C7, C8: LCSC (none) -> C1711
- D2: LCSC (none) -> C6807778
- D3, D4: LCSC (none) -> C3018534
- F1: LCSC (none) -> C151075
- J11, J12: LCSC (none) -> C3820334
- J14, J15: LCSC (none) -> C5441017
- L3, L4: LCSC (none) -> C6577597
- R4, R5: value 2k94 -> 3k; LCSC (none) -> C17661
- R6, R8: value 17k8 -> 18k; LCSC (none) -> C17506
- R7, R9: LCSC (none) -> C4310
- U7: LCSC (none) -> C5276750
- U8, U9: LCSC (none) -> C1355343
Changed lines of the file:
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@@
   (title_block
     (title "Tandem Leveller Controller")
-    (date "2025-02-22")
+    (date "2025-03-11")
     (rev "V1.0")
     (company "(C) andy@britishideas.com 2025")
@@
       (effects (font (size 1.27 1.27)) (justify left))
     )
-    (property "Value" "17k8" (at 217.17 63.5 0)
+    (property "Value" "18k" (at 217.17 63.5 0)
       (effects (font (size 1.27 1.27)) (justify left))
     )
@@
     )
     (property "Datasheet" "~" (at 214.63 62.23 0)
+      (effects (font (size 1.27 1.27)) hide)
+    )
+    (property "LCSC" "C17506" (at 214.63 62.23 0)
       (effects (font (size 1.27 1.27)) hide)
     )
@@
       (effects (font (size 1.27 1.27)) hide)
     )
+    (property "LCSC" "C5276750" (at 100.965 93.98 0)
+      (effects (font (size 1.27 1.27)) hide)
+    )
     (pin "1")
     (pin "5")
@@
       (effects (font (size 1.27 1.27)) (justify left))
     )
-    (property "Value" "2k94" (at 173.99 130.175 0)
+    (property "Value" "3k" (at 173.99 130.175 0)
       (effects (font (size 1.27 1.27)) (justify left))
     )
@@
       (effects (font (size 1.27 1.27)) hide)
     )
+    (property "LCSC" "C17661" (at 171.45 128.905 0)
+      (effects (font (size 1.27 1.27)) hide)
+    )
     (pin "1")
     (pin "2")
@@
       (effects (font (size 1.27 1.27)) hide)
     )
+    (property "LCSC" "" (at 123.825 96.52 0)
+      (effects (font (size 1.27 1.27)) hide)
+    )
     (pin "1")
     (pin "2")
@@
       (effects (font (size 1.27 1.27)) hide)
     )
+    (property "LCSC" "C3340" (at 131.445 101.6 0)
+      (effects (font (size 1.27 1.27)) hide)
+    )
     (pin "1")
     (pin "2")
@@
     )
     (property "Datasheet" "~" (at 207.645 113.665 0)
+      (effects (font (size 1.27 1.27)) hide)
+    )
+    (property "LCSC" "C3018534" (at 207.645 113.665 0)
       (effects (font (size 1.27 1.27)) hide)
     )
@@
       (effects (font (size 1.27 1.27)) hide)
     )
+    (property "LCSC" "C5441017" (at 243.84 59.69 0)
+      (effects (font (size 1.27 1.27)) hide)
+    )
     (pin "2")
     (pin "1")
@@
     )
     (property "Datasheet" "~" (at 194.945 52.07 0)
+      (effects (font (size 1.27 1.27)) hide)
+    )
+    (property "LCSC" "C6577597" (at 194.945 52.07 0)
       (effects (font (size 1.27 1.27)) hide)
     )
@@
       (effects (font (size 1.27 1.27)) hide)
     )
+    (property "LCSC" "C3820334" (at 27.305 93.98 0)
+      (effects (font (size 1.27 1.27)) hide)
+    )
     (pin "2")
     (pin "1")
@@
       (effects (font (size 1.27 1.27)) hide)
     )
-    (property "Field5" "" (at 224.79 73.025 0)
+    (property "LCSC" "C1984785" (at 224.79 73.025 0)
       (effects (font (size 1.27 1.27)) hide)
     )
@@
       (effects (font (size 1.27 1.27)) hide)
     )
+    (property "LCSC" "C5441017" (at 243.84 116.205 0)
+      (effects (font (size 1.27 1.27)) hide)
+    )
     (pin "2")
     (pin "1")
@@
       (effects (font (size 1.27 1.27)) hide)
     )
+    (property "LCSC" "C6577597" (at 194.945 108.585 0)
+      (effects (font (size 1.27 1.27)) hide)
+    )
     (pin "1")
     (pin "2")
@@
     )
     (property "Datasheet" "" (at 179.07 130.175 0)
+      (effects (font (size 1.27 1.27)) hide)
+    )
+    (property "LCSC" "C1355343" (at 179.07 130.175 0)
       (effects (font (size 1.27 1.27)) hide)
     )
@@
       (effects (font (size 1.27 1.27)) hide)
     )
+    (property "LCSC" "C4310" (at 214.63 73.025 0)
+      (effects (font (size 1.27 1.27)) hide)
+    )
     (pin "1")
     (pin "2")
@@
       (effects (font (size 1.27 1.27)) hide)
     )
+    (property "LCSC" "C1711" (at 171.45 138.43 0)
+      (effects (font (size 1.27 1.27)) hide)
+    )
     (pin "2")
     (pin "1")
@@
     )
     (property "manf#" "1729034" (at 103.505 139.065 0)
+      (effects (font (size 1.27 1.27)) hide)
+    )
+    (property "LCSC" "" (at 103.505 139.065 0)
       (effects (font (size 1.27 1.27)) hide)
     )
@@
       (effects (font (size 1.27 1.27)) hide)
     )
+    (property "LCSC" "C340733" (at 163.195 60.96 0)
+      (effects (font (size 1.27 1.27)) hide)
+    )
     (pin "1")
     (pin "2")
@@
       (effects (font (size 1.27 1.27)) (justify left))
     )
-    (property "Value" "2k94" (at 173.99 73.66 0)
+    (property "Value" "3k" (at 173.99 73.66 0)
       (effects (font (size 1.27 1.27)) (justify left))
     )
@@
       (effects (font (size 1.27 1.27)) hide)
     )
+    (property "LCSC" "C17661" (at 171.45 72.39 0)
+      (effects (font (size 1.27 1.27)) hide)
+    )
     (pin "1")
     (pin "2")
@@
       (effects (font (size 1.27 1.27)) hide)
     )
+    (property "LCSC" "C6807778" (at 118.11 101.6 0)
+      (effects (font (size 1.27 1.27)) hide)
+    )
     (pin "1")
     (pin "2")
@@
       (effects (font (size 1.27 1.27)) hide)
     )
+    (property "LCSC" "C340733" (at 163.195 117.475 0)
+      (effects (font (size 1.27 1.27)) hide)
+    )
     (pin "1")
     (pin "2")
@@
     )
     (property "Datasheet" "" (at 179.07 73.66 0)
+      (effects (font (size 1.27 1.27)) hide)
+    )
+    (property "LCSC" "C1355343" (at 179.07 73.66 0)
       (effects (font (size 1.27 1.27)) hide)
     )
@@
       (effects (font (size 1.27 1.27)) hide)
     )
+    (property "LCSC" "C1711" (at 171.45 81.915 0)
+      (effects (font (size 1.27 1.27)) hide)
+    )
     (pin "2")
     (pin "1")
@@
       (effects (font (size 1.27 1.27)) hide)
     )
+    (property "LCSC" "C3018534" (at 207.645 57.15 0)
+      (effects (font (size 1.27 1.27)) hide)
+    )
     (pin "1")
     (pin "2")
@@
       (effects (font (size 1.27 1.27)) (justify left))
     )
-    (property "Value" "17k8" (at 217.17 120.015 0)
+    (property "Value" "18k" (at 217.17 120.015 0)
       (effects (font (size 1.27 1.27)) (justify left))
     )
@@
     )
     (property "Datasheet" "~" (at 214.63 118.745 0)
+      (effects (font (size 1.27 1.27)) hide)
+    )
+    (property "LCSC" "C17506" (at 214.63 118.745 0)
       (effects (font (size 1.27 1.27)) hide)
     )
@@
       (effects (font (size 1.27 1.27)) hide)
     )
+    (property "LCSC" "C3820334" (at 49.53 86.36 0)
+      (effects (font (size 1.27 1.27)) hide)
+    )
     (pin "2")
     (pin "1")
@@
       (effects (font (size 1.27 1.27)) hide)
     )
+    (property "LCSC" "C50456" (at 76.835 97.155 0)
+      (effects (font (size 1.27 1.27)) hide)
+    )
     (pin "1")
     (pin "2")
@@
       (effects (font (size 1.27 1.27)) hide)
     )
+    (property "LCSC" "C1984785" (at 224.79 129.54 0)
+      (effects (font (size 1.27 1.27)) hide)
+    )
     (pin "1")
     (pin "2")
@@
       (effects (font (size 1.27 1.27)))
     )
+    (property "LCSC" "C151075" (at 67.945 91.44 0)
+      (effects (font (size 1.27 1.27)) hide)
+    )
     (pin "2")
     (pin "1")
@@
       (effects (font (size 1.27 1.27)) hide)
     )
+    (property "LCSC" "C4310" (at 214.63 129.54 0)
+      (effects (font (size 1.27 1.27)) hide)
+    )
