File: Electronics/Controller/Power.kicad_sch (KiCad schematic)
At the start: 29 parts, among them J11 TRACTOR BATTERY, J12 PWR SWITCH, J13 VALVE POWER, J14 TABLET 1 PWR, J15 TABLET 2 PWR, U7 LM2596S-5, U8 LM2587S-ADJ/NOPB, U9 LM2587S-ADJ/NOPB

Commit message: Added inductor part number.
Parts:
- L2: manf# (none) -> AWVS00808040330M00
Changed lines of the file:
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@@
+      (effects (font (size 1.27 1.27)) hide)
+    )
+    (property "manf#" "AWVS00808040330M00" (at 123.825 96.52 90)
       (effects (font (size 1.27 1.27)) hide)
     )

Commit message: Changed four way screw block, USB type A connectors, 33uH inductor and 24MHz crystal to use parts that JLCPCB has in stock.
Parts:
- C5, C6: value 100u -> 1729034
- J13: LCSC (none) -> C7032066; manf# 1729034 -> 691137710004
- L2: footprint Britishideas:Chilisin_Power_Inductor_AWVS_808040 -> Britishideas:MWSA0603S-330MT; LCSC (none) -> C408454; manf# AWVS00808040330M00 -> MWSA0603S-330MT
Changed lines of the file:
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@@
   (title_block
     (title "Tandem Leveller Controller")
-    (date "2025-03-13")
+    (date "2025-03-18")
     (rev "V1.0")
     (company "(C) andy@britishideas.com 2025")
@@
       (effects (font (size 1.27 1.27)))
     )
-    (property "Footprint" "Britishideas:Chilisin_Power_Inductor_AWVS_808040" (at 123.825 96.52 0)
+    (property "Footprint" "Britishideas:MWSA0603S-330MT" (at 123.825 96.52 0)
       (effects (font (size 1.27 1.27)) hide)
     )
@@
       (effects (font (size 1.27 1.27)) hide)
     )
-    (property "LCSC" "" (at 123.825 96.52 0)
-      (effects (font (size 1.27 1.27)) hide)
-    )
-    (property "manf#" "AWVS00808040330M00" (at 123.825 96.52 90)
+    (property "LCSC" "C408454" (at 123.825 96.52 0)
+      (effects (font (size 1.27 1.27)) hide)
+    )
+    (property "manf#" "MWSA0603S-330MT" (at 123.825 96.52 90)
       (effects (font (size 1.27 1.27)) hide)
     )
@@
       (effects (font (size 1.27 1.27)) hide)
     )
-    (property "manf#" "1729034" (at 103.505 139.065 0)
-      (effects (font (size 1.27 1.27)) hide)
-    )
-    (property "LCSC" "" (at 103.505 139.065 0)
+    (property "manf#" "691137710004" (at 103.505 139.065 0)
+      (effects (font (size 1.27 1.27)) hide)
+    )
+    (property "LCSC" "C7032066" (at 103.505 139.065 0)
       (effects (font (size 1.27 1.27)) hide)
     )
@@
       (effects (font (size 1.27 1.27)) (justify left))
     )
-    (property "Value" "100u" (at 166.37 61.341 0)
+    (property "Value" "1729034" (at 166.37 61.341 0)
       (effects (font (size 1.27 1.27)) (justify left))
     )
@@
       (effects (font (size 1.27 1.27)) (justify left))
     )
-    (property "Value" "100u" (at 166.37 117.856 0)
-      (effects (font (size 1.27 1.27)) (justify left))
-    )
+    (property "Value" "1729034" (at 166.37 117.856 0)
+      (effects (font (size 1.27 1.27)) (justify left))
+    )

Commit message: Changed tablet PSU inductors.
Parts:
- L3, L4: value IHLP6767DZER470M11 -> MWSA1206S-470MT; footprint Britishideas:IHLP6767DZER470M11 -> Britishideas:MWSA1206S-470MT; LCSC C6577597 -> C408531; manf# (none) -> MWSA1206S-470MT
Changed lines of the file:
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@@
       (effects (font (size 1.27 1.27)))
     )
-    (property "Value" "IHLP6767DZER470M11" (at 194.945 50.165 90)
+    (property "Value" "MWSA1206S-470MT" (at 194.945 50.165 90)
       (effects (font (size 1.27 1.27)))
     )
-    (property "Footprint" "Britishideas:IHLP6767DZER470M11" (at 194.945 52.07 0)
+    (property "Footprint" "Britishideas:MWSA1206S-470MT" (at 194.945 52.07 0)
       (effects (font (size 1.27 1.27)) hide)
     )
@@
       (effects (font (size 1.27 1.27)) hide)
     )
-    (property "LCSC" "C6577597" (at 194.945 52.07 0)
+    (property "LCSC" "C408531" (at 194.945 52.07 0)
+      (effects (font (size 1.27 1.27)) hide)
+    )
+    (property "manf#" "MWSA1206S-470MT" (at 194.945 52.07 90)
       (effects (font (size 1.27 1.27)) hide)
     )
@@
       (effects (font (size 1.27 1.27)))
     )
-    (property "Value" "IHLP6767DZER470M11" (at 194.945 106.68 90)
+    (property "Value" "MWSA1206S-470MT" (at 194.945 106.68 90)
       (effects (font (size 1.27 1.27)))
     )
-    (property "Footprint" "Britishideas:IHLP6767DZER470M11" (at 194.945 108.585 0)
+    (property "Footprint" "Britishideas:MWSA1206S-470MT" (at 194.945 108.585 0)
       (effects (font (size 1.27 1.27)) hide)
     )
@@
       (effects (font (size 1.27 1.27)) hide)
     )
-    (property "LCSC" "C6577597" (at 194.945 108.585 0)
+    (property "LCSC" "C408531" (at 194.945 108.585 0)
       (effects (font (size 1.27 1.27)) hide)
     )
+    (property "manf#" "MWSA1206S-470MT" (at 194.945 108.585 90)
+      (effects (font (size 1.27 1.27)) hide)
+    )
