File: Electronics/Controller/Slave Tablet.kicad_sch (KiCad schematic)
At the start: 13 parts, among them J16 SLAVE TABLET, U14 FT232RL, U15 FT232RL

Commit message: Changed four way screw block, USB type A connectors, 33uH inductor and 24MHz crystal to use parts that JLCPCB has in stock.
Parts:
- FB1: value MI0805K400R-10 -> PZ2012D800-3R0TF; LCSC (none) -> C12389; manf# MI0805K400R-10 -> PZ2012D800-3R0TF
Changed lines of the file:
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@@
   (title_block
     (title "Tandem Leveller Controller")
-    (date "2025-03-13")
+    (date "2025-03-18")
     (rev "V1.0")
     (company "(C) andy@britishideas.com 2025")
@@
       (effects (font (size 1.27 1.27)) (justify left))
     )
-    (property "Value" "MI0805K400R-10" (at 226.06 69.1769 0)
+    (property "Value" "PZ2012D800-3R0TF" (at 226.06 69.1769 0)
       (effects (font (size 1.27 1.27)) (justify left))
     )
@@
       (effects (font (size 1.27 1.27)) hide)
     )
-    (property "manf#" "MI0805K400R-10" (at 222.885 67.945 0)
-      (effects (font (size 1.27 1.27)) hide)
-    )
-    (property "LCSC" "" (at 222.885 67.945 0)
-      (effects (font (size 1.27 1.27)) hide)
-    )
+    (property "manf#" "PZ2012D800-3R0TF" (at 222.885 67.945 0)
+      (effects (font (size 1.27 1.27)) hide)
+    )
+    (property "LCSC" "C12389" (at 222.885 67.945 0)
+      (effects (font (size 1.27 1.27)) hide)
+    )
