File: Electronics/Controller/USB Hub.kicad_sch (KiCad schematic)
At the start: 45 parts, among them J17 MASTER TABLET, J18 292303-7, J19 292303-7, U16 USB2517, U17 MIC2026-1YM, Y1 FA-238 24.0000MD30X-W5

Commit message: Changed four way screw block, USB type A connectors, 33uH inductor and 24MHz crystal to use parts that JLCPCB has in stock.
Parts:
- C44, C45: value 100u -> 1729034
- FB2: value MI0805K400R-10 -> PZ2012D800-3R0TF; LCSC (none) -> C12389; manf# MI0805K400R-10 -> PZ2012D800-3R0TF
- J18, J19: value 292303-7 -> 292303-1; footprint Connector_USB:USB_A_TE_292303-7_Horizontal -> Britishideas:292303-1; LCSC (none) -> C86461; manf# (none) -> 292303-1
- Y1: value FA-238 24.0000MD30X-W5 -> CF4024M00012; footprint EmSA:FA-238 -> Britishideas:FA-238; LCSC (none) -> C5765976; manf# FA-238V 12.0000MB-W3 -> CF4024M00012
Changed lines of the file:
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@@
   (title_block
     (title "Tandem Leveller Controller")
-    (date "2025-03-13")
+    (date "2025-03-18")
     (rev "V1.0")
     (company "(C) andy@britishideas.com 2025")
@@
       (effects (font (size 1.27 1.27)) (justify left))
     )
-    (property "Value" "MI0805K400R-10" (at 53.975 26.6319 0)
+    (property "Value" "PZ2012D800-3R0TF" (at 53.975 26.6319 0)
       (effects (font (size 1.27 1.27)) (justify left))
     )
@@
       (effects (font (size 1.27 1.27)) hide)
     )
-    (property "manf#" "MI0805K400R-10" (at 57.15 25.4 0)
-      (effects (font (size 1.27 1.27)) hide)
-    )
-    (property "LCSC" "" (at 57.15 25.4 0)
+    (property "manf#" "PZ2012D800-3R0TF" (at 57.15 25.4 0)
+      (effects (font (size 1.27 1.27)) hide)
+    )
+    (property "LCSC" "C12389" (at 57.15 25.4 0)
       (effects (font (size 1.27 1.27)) hide)
     )
@@
       (effects (font (size 1.27 1.27)) (justify left))
     )
-    (property "Value" "100u" (at 271.78 73.025 0)
+    (property "Value" "1729034" (at 271.78 73.025 0)
       (effects (font (size 1.27 1.27)) (justify left))
     )
@@
       (effects (font (size 1.27 1.27)) (justify right))
     )
-    (property "Value" "292303-7" (at 248.92 139.065 0)
+    (property "Value" "292303-1" (at 248.92 139.065 0)
       (effects (font (size 1.27 1.27)) (justify right))
     )
-    (property "Footprint" "Connector_USB:USB_A_TE_292303-7_Horizontal" (at 238.125 139.065 0)
+    (property "Footprint" "Britishideas:292303-1" (at 238.125 139.065 0)
       (effects (font (size 1.27 1.27)) hide)
     )
@@
       (effects (font (size 1.27 1.27)) hide)
     )
-    (property "LCSC" "" (at 241.935 137.795 0)
+    (property "LCSC" "C86461" (at 241.935 137.795 0)
+      (effects (font (size 1.27 1.27)) hide)
+    )
+    (property "manf#" "292303-1" (at 241.935 137.795 0)
       (effects (font (size 1.27 1.27)) hide)
     )
@@
       (effects (font (size 1.27 1.27)))
     )
-    (property "Value" "FA-238 24.0000MD30X-W5" (at 27.305 93.345 90)
-      (effects (font (size 1.27 1.27)))
-    )
-    (property "Footprint" "EmSA:FA-238" (at 36.195 100.33 0)
+    (property "Value" "CF4024M00012" (at 27.305 93.345 90)
+      (effects (font (size 1.27 1.27)))
+    )
+    (property "Footprint" "Britishideas:FA-238" (at 36.195 100.33 0)
       (effects (font (size 1.27 1.27)) hide)
     )
@@
       (effects (font (size 1.27 1.27)) hide)
     )
-    (property "manf#" "FA-238V 12.0000MB-W3" (at 36.195 100.33 0)
-      (effects (font (size 1.27 1.27)) hide)
-    )
-    (property "LCSC" "" (at 36.195 100.33 0)
+    (property "manf#" "CF4024M00012" (at 36.195 100.33 0)
+      (effects (font (size 1.27 1.27)) hide)
+    )
+    (property "LCSC" "C5765976" (at 36.195 100.33 0)
       (effects (font (size 1.27 1.27)) hide)
     )
@@
   (symbol (lib_id "Connector:USB_A") (at 241.935 100.33 0) (mirror y) (unit 1)
     (in_bom yes) (on_board yes) (dnp no) (fields_autoplaced)
-    (property "Reference" "J18" (at 248.285 99.06 0)
+    (property "Reference" "J18" (at 248.92 99.06 0)
       (effects (font (size 1.27 1.27)) (justify right))
     )
-    (property "Value" "292303-7" (at 248.285 101.6 0)
+    (property "Value" "292303-1" (at 248.92 101.6 0)
       (effects (font (size 1.27 1.27)) (justify right))
     )
-    (property "Footprint" "Connector_USB:USB_A_TE_292303-7_Horizontal" (at 238.125 101.6 0)
+    (property "Footprint" "Britishideas:292303-1" (at 238.125 101.6 0)
       (effects (font (size 1.27 1.27)) hide)
     )
@@
       (effects (font (size 1.27 1.27)) hide)
     )
-    (property "LCSC" "" (at 241.935 100.33 0)
+    (property "LCSC" "C86461" (at 241.935 100.33 0)
+      (effects (font (size 1.27 1.27)) hide)
+    )
+    (property "manf#" "292303-1" (at 241.935 100.33 0)
       (effects (font (size 1.27 1.27)) hide)
     )
@@
       (effects (font (size 1.27 1.27)) (justify left))
     )
-    (property "Value" "100u" (at 260.35 73.025 0)
-      (effects (font (size 1.27 1.27)) (justify left))
-    )
+    (property "Value" "1729034" (at 260.35 73.025 0)
+      (effects (font (size 1.27 1.27)) (justify left))
+    )
