File: Electronics/GPS IMU Simulator/GPS IMU Simulator/CAN.kicad_sch (KiCad schematic)
At the start: 9 parts, among them J2 TERM, J4 CAN BUS, U2 TJA1462ATK-0Z, U3 PESD2CANFD24V-TR

Commit message: Added 4.7uF caps to FT232RL on controller.
Parts:
- C1, C2: LCSC (none) -> C1711
- J2: LCSC (none) -> C7494857
- J4: LCSC (none) -> C157993
- L1: LCSC (none) -> C95572
- R2: LCSC (none) -> C17414
- R3: LCSC (none) -> C17437
- U2: LCSC (none) -> C3229259
- U3: LCSC (none) -> C552486
Changed lines of the file:
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@@
+      (effects (font (size 1.27 1.27)) hide)
+    )
+    (property "LCSC" "C1711" (at 69.215 135.255 0)
       (effects (font (size 1.27 1.27)) hide)
     )
@@
     )
     (property "Datasheet" "~" (at 97.79 105.41 0)
+      (effects (font (size 1.27 1.27)) hide)
+    )
+    (property "LCSC" "C17414" (at 97.79 105.41 0)
       (effects (font (size 1.27 1.27)) hide)
     )
@@
       (effects (font (size 1.27 1.27)) hide)
     )
+    (property "LCSC" "C157993" (at 224.155 93.98 0)
+      (effects (font (size 1.27 1.27)) hide)
+    )
     (pin "2")
     (pin "5")
@@
     )
     (property "manf#" "TJA1462ATK/0Z" (at 76.2 86.36 0)
+      (effects (font (size 1.27 1.27)) hide)
+    )
+    (property "LCSC" "C3229259" (at 68.58 101.6 0)
       (effects (font (size 1.27 1.27)) hide)
     )
@@
       (effects (font (size 1.27 1.27)) hide)
     )
+    (property "LCSC" "C552486" (at 139.065 109.22 0)
+      (effects (font (size 1.27 1.27)) hide)
+    )
     (pin "1")
     (pin "2")
@@
       (effects (font (size 1.27 1.27)) hide)
     )
+    (property "LCSC" "C95572" (at 119.38 96.52 0)
+      (effects (font (size 1.27 1.27)) hide)
+    )
     (pin "1")
     (pin "2")
@@
       (effects (font (size 1.27 1.27)) hide)
     )
+    (property "LCSC" "C1711" (at 80.01 135.255 0)
+      (effects (font (size 1.27 1.27)) hide)
+    )
     (pin "1")
     (pin "2")
@@
     )
     (property "Datasheet" "~" (at 173.99 77.47 0)
+      (effects (font (size 1.27 1.27)) hide)
+    )
+    (property "LCSC" "C7494857" (at 173.99 77.47 0)
       (effects (font (size 1.27 1.27)) hide)
     )
@@
       (effects (font (size 1.27 1.27)) hide)
     )
+    (property "LCSC" "C17437" (at 173.99 87.63 0)
+      (effects (font (size 1.27 1.27)) hide)
+    )
