File: Electronics/GPS IMU Simulator/GPS IMU Simulator/GNSS.kicad_sch (KiCad schematic)
At the start: 1 part, among them J3 GPS SIM

Commit message: Added 4.7uF caps to FT232RL on controller.
Parts:
- J3: LCSC (none) -> C157974
Changed lines of the file:
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@@
     (comment 2 "Provided as-is, no warranty express or implied. Use at your own risk")
   )
-  (wire (pts (xy 127 51.435) (xy 146.05 51.435))
+  (wire (pts (xy 127 88.9) (xy 146.05 88.9))
     (stroke (width 0) (type default))
   )
@@
     (stroke (width 0) (type default))
   )
-  (wire (pts (xy 143.51 113.03) (xy 143.51 48.895))
+  (wire (pts (xy 143.51 113.03) (xy 143.51 86.36))
     (stroke (width 0) (type default))
   )
@@
     (stroke (width 0) (type default))
   )
-  (wire (pts (xy 127 48.895) (xy 143.51 48.895))
+  (wire (pts (xy 127 86.36) (xy 143.51 86.36))
     (stroke (width 0) (type default))
   )
@@
     (stroke (width 0) (type default))
   )
-  (wire (pts (xy 146.05 115.57) (xy 146.05 51.435))
+  (wire (pts (xy 146.05 115.57) (xy 146.05 88.9))
     (stroke (width 0) (type default))
   )
@@
     (effects (font (size 1.27 1.27)) (justify right))
   )
-  (hierarchical_label "GNSS_TRACTOR_RX" (shape output) (at 127 51.435 180) (fields_autoplaced)
+  (hierarchical_label "GNSS_TRACTOR_RX" (shape output) (at 127 88.9 180) (fields_autoplaced)
     (effects (font (size 1.27 1.27)) (justify right))
   )
@@
     (effects (font (size 1.27 1.27)) (justify right))
   )
-  (hierarchical_label "GNSS_TRACTOR_TX" (shape input) (at 127 48.895 180) (fields_autoplaced)
+  (hierarchical_label "GNSS_TRACTOR_TX" (shape input) (at 127 86.36 180) (fields_autoplaced)
     (effects (font (size 1.27 1.27)) (justify right))
   )
@@
       (effects (font (size 1.27 1.27)) hide)
     )
+    (property "LCSC" "C157974" (at 128.905 120.65 0)
+      (effects (font (size 1.27 1.27)) hide)
+    )
