File: Electronics/GPS IMU Simulator/GPS IMU Simulator/GPS IMU Simulator.kicad_sch (KiCad schematic)
At the start: 5 parts, among them J1 BUTTON 1, J11 Conn_01x02, J9 JOYSTICK 1, U1 TEENSY 4.0

Commit message: Added 4.7uF caps to FT232RL on controller.
Parts:
- J1: LCSC (none) -> C131334
- J11: LCSC (none) -> C7494857
- J9: LCSC (none) -> C157993
- R1: LCSC (none) -> C17414
- U1: LCSC (none) -> C2897377
Changed lines of the file:
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@@
+      (effects (font (size 1.27 1.27)) hide)
+    )
+    (property "LCSC" "C17414" (at 68.58 61.595 0)
       (effects (font (size 1.27 1.27)) hide)
     )
@@
       (effects (font (size 1.27 1.27)) hide)
     )
+    (property "LCSC" "C7494857" (at 149.225 60.325 0)
+      (effects (font (size 1.27 1.27)) hide)
+    )
     (pin "1")
     (pin "2")
@@
     )
     (property "manf#" "B5B-PH-K-S" (at 57.15 109.855 0)
+      (effects (font (size 1.27 1.27)) hide)
+    )
+    (property "LCSC" "C157993" (at 57.15 109.855 0)
       (effects (font (size 1.27 1.27)) hide)
     )
@@
     )
     (property "Datasheet" "" (at 133.985 190.5 0)
+      (effects (font (size 1.27 1.27)) hide)
+    )
+    (property "LCSC" "C2897377" (at 133.985 190.5 0)
       (effects (font (size 1.27 1.27)) hide)
     )
@@
       (effects (font (size 1.27 1.27)) hide)
     )
+    (property "LCSC" "C131334" (at 52.07 71.12 0)
+      (effects (font (size 1.27 1.27)) hide)
+    )

Commit message: Removed JLCPCB part numbers for Teensy and BNO085 connectors. Added JLCPCB part number for 4.7uF capacitor. Generated JLCPCB manufacturing files for all boards.
Parts:
- U1: LCSC C2897377 -> (none)
Changed lines of the file:
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@@
       (effects (font (size 1.27 1.27)) hide)
     )
-    (property "LCSC" "C2897377" (at 133.985 190.5 0)
+    (property "LCSC" "" (at 133.985 190.5 0)
       (effects (font (size 1.27 1.27)) hide)
     )

Commit message: Added fiducials to all boards.
Parts:
- added FID1, FID2, FID3: Fiducial, Fiducial:Fiducial_0.5mm_Mask1mm, symbol Mechanical:Fiducial
Changed lines of the file:
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@@
   (title_block
     (title "GPS and IMU Simulator")
-    (date "2025-03-04")
+    (date "2025-03-13")
     (rev "V1.0")
     (company "(C) andy@britishideas.com 2025")
@@
     )
   )
+  (symbol (lib_id "Mechanical:Fiducial") (at 163.83 186.69 0) (unit 1)
+    (in_bom yes) (on_board yes) (dnp no) (fields_autoplaced)
+    (property "Reference" "FID1" (at 166.37 185.42 0)
+      (effects (font (size 1.27 1.27)) (justify left))
+    )
+    (property "Value" "Fiducial" (at 166.37 187.96 0)
+      (effects (font (size 1.27 1.27)) (justify left))
+    )
+    (property "Footprint" "Fiducial:Fiducial_0.5mm_Mask1mm" (at 163.83 186.69 0)
+      (effects (font (size 1.27 1.27)) hide)
+    )
+    (property "Datasheet" "~" (at 163.83 186.69 0)
+      (effects (font (size 1.27 1.27)) hide)
+    )
+    (instances
+      (project "GPS IMU Simulator"
+        (path "/1f585cd8-3c8f-431c-b995-1ddab1655b89"
+          (reference "FID1") (unit 1)
+        )
+      )
+    )
+  )
   (symbol (lib_id "power:+5V") (at 73.025 55.245 0) (unit 1)
     (in_bom yes) (on_board yes) (dnp no)
@@
         (path "/1f585cd8-3c8f-431c-b995-1ddab1655b89"
           (reference "#PWR05") (unit 1)
+        )
+      )
+    )
+  )
+  (symbol (lib_id "Mechanical:Fiducial") (at 151.765 186.69 0) (unit 1)
+    (in_bom yes) (on_board yes) (dnp no) (fields_autoplaced)
+    (property "Reference" "FID2" (at 154.305 185.42 0)
+      (effects (font (size 1.27 1.27)) (justify left))
+    )
+    (property "Value" "Fiducial" (at 154.305 187.96 0)
+      (effects (font (size 1.27 1.27)) (justify left))
+    )
+    (property "Footprint" "Fiducial:Fiducial_0.5mm_Mask1mm" (at 151.765 186.69 0)
+      (effects (font (size 1.27 1.27)) hide)
+    )
+    (property "Datasheet" "~" (at 151.765 186.69 0)
+      (effects (font (size 1.27 1.27)) hide)
+    )
+    (instances
+      (project "GPS IMU Simulator"
+        (path "/1f585cd8-3c8f-431c-b995-1ddab1655b89"
+          (reference "FID2") (unit 1)
         )
       )
@@
         )
       )
+    )
+  )
+  (symbol (lib_id "Mechanical:Fiducial") (at 139.7 186.69 0) (unit 1)
+    (in_bom yes) (on_board yes) (dnp no) (fields_autoplaced)
+    (property "Reference" "FID3" (at 142.24 185.42 0)
+      (effects (font (size 1.27 1.27)) (justify left))
+    )
+    (property "Value" "Fiducial" (at 142.24 187.96 0)
+      (effects (font (size 1.27 1.27)) (justify left))
+    )
+    (property "Footprint" "Fiducial:Fiducial_0.5mm_Mask1mm" (at 139.7 186.69 0)
+      (effects (font (size 1.27 1.27)) hide)
+    )
+    (property "Datasheet" "~" (at 139.7 186.69 0)
+      (effects (font (size 1.27 1.27)) hide)
+    )
+    (instances
+      (project "GPS IMU Simulator"
+        (path "/1f585cd8-3c8f-431c-b995-1ddab1655b89"
+          (reference "FID3") (unit 1)
+        )
+      )
