File: Electronics/IMU/CAN.kicad_sch (KiCad schematic)
At the start: 10 parts, among them J2 TERM, J3 CAN BUS, J4 CAN BUS, U3 TJA1462ATK-0Z, U4 PESD2CANFD24V-TR

Commit message: Completed first attempt at GPS/IMU simulator.
Parts:
- C1, C2: LCSC (none) -> C1711
- J3, J4: LCSC (none) -> C157993
- L1: LCSC (none) -> C95572
- R1: LCSC (none) -> C17414
- R2: LCSC (none) -> C17437
- U3: LCSC (none) -> C3229259
- U4: LCSC (none) -> C552486
Changed lines of the file:
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@@
+      (effects (font (size 1.27 1.27)) hide)
+    )
+    (property "LCSC" "C17437" (at 176.53 83.82 0)
       (effects (font (size 1.27 1.27)) hide)
     )
@@
       (effects (font (size 1.27 1.27)) hide)
     )
+    (property "LCSC" "C157993" (at 243.84 90.17 0)
+      (effects (font (size 1.27 1.27)) hide)
+    )
     (pin "2")
     (pin "5")
@@
     )
     (property "manf#" "TJA1462ATK/0Z" (at 78.74 82.55 0)
+      (effects (font (size 1.27 1.27)) hide)
+    )
+    (property "LCSC" "C3229259" (at 71.12 97.79 0)
       (effects (font (size 1.27 1.27)) hide)
     )
@@
       (effects (font (size 1.27 1.27)) hide)
     )
+    (property "LCSC" "C552486" (at 141.605 105.41 0)
+      (effects (font (size 1.27 1.27)) hide)
+    )
     (pin "1")
     (pin "2")
@@
       (effects (font (size 1.27 1.27)) hide)
     )
+    (property "LCSC" "C1711" (at 82.55 131.445 0)
+      (effects (font (size 1.27 1.27)) hide)
+    )
     (pin "1")
     (pin "2")
@@
     )
     (property "manf#" "ACT1210-510-2P-TL00" (at 121.92 92.71 0)
+      (effects (font (size 1.27 1.27)) hide)
+    )
+    (property "LCSC" "C95572" (at 121.92 92.71 0)
       (effects (font (size 1.27 1.27)) hide)
     )
@@
     )
     (property "Datasheet" "~" (at 71.755 131.445 0)
+      (effects (font (size 1.27 1.27)) hide)
+    )
+    (property "LCSC" "C1711" (at 71.755 131.445 0)
       (effects (font (size 1.27 1.27)) hide)
     )
@@
       (effects (font (size 1.27 1.27)) hide)
     )
+    (property "LCSC" "C157993" (at 243.84 105.41 0)
+      (effects (font (size 1.27 1.27)) hide)
+    )
     (pin "2")
     (pin "5")
@@
       (effects (font (size 1.27 1.27)) hide)
     )
+    (property "LCSC" "C17414" (at 100.33 101.6 0)
+      (effects (font (size 1.27 1.27)) hide)
+    )

Commit message: Added 4.7uF caps to FT232RL on controller.
Parts:
- J2: LCSC (none) -> C7494857
Changed lines of the file:
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@@
+      (effects (font (size 1.27 1.27)) hide)
+    )
+    (property "LCSC" "C7494857" (at 176.53 73.66 0)
       (effects (font (size 1.27 1.27)) hide)
     )
@@
       (effects (font (size 1.27 1.27)) hide)
     )
+    (property "manf#" "" (at 100.33 101.6 0)
+      (effects (font (size 1.27 1.27)) hide)
+    )
