File: Electronics/IMU/IMU.kicad_pcb (KiCad board)
At the start: 2 copper layers, 52 x 59 mm, 13 parts, among them J1 Conn_01x02, J2 TERM, J3 CAN BUS, J4 CAN BUS, U1 TEENSY 4.0, U2 Adafruit BNO085, U3 TJA1462ATK-0Z, U4 PESD2CANFD24V-TR

Commit message: Working on IMU PCB.
Routing:
- net +5V: track 0.00 -> 76.0 mm, vias 0 -> 2
- net Net-(U1-GPIO12_MISO): track 0.00 -> 45.4 mm
- net Net-(U1-GPIO13_SCK_CRX1): track 0.00 -> 29.1 mm
- net Net-(U1-GPIO16_RX4_SCL1): track 0.00 -> 28.0 mm
- net Net-(U1-GPIO11_MOSI): track 0.00 -> 26.5 mm
- net Net-(U1-GPIO10_CS): track 0.00 -> 26.5 mm
- net /CAN/CAN_H: track 0.00 -> 24.4 mm, vias 0 -> 2
- net /CAN/CAN_L: track 0.00 -> 20.2 mm
- net /CAN/CAN_RX: track 0.00 -> 13.7 mm, vias 0 -> 2
- net /CAN/CAN_TX: track 0.00 -> 12.9 mm, vias 0 -> 2
- net Net-(U1-GPIO15_RX3): track 0.00 -> 10.1 mm
- net +12V: track 0.00 -> 6.20 mm
- net Net-(J1-Pin_1): track 0.00 -> 4.05 mm
- net Net-(U3-CANH): track 0.00 -> 3.79 mm
- net Net-(J2-Pin_1): track 0.00 -> 3.72 mm
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Other:
- board text added: "EN"

Commit message: Completed first attempt at GPS/IMU simulator.
Changed lines of the file:
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@@
       (outputformat 1)
       (mirror false)
-      (drillshape 1)
+      (drillshape 0)
       (scaleselection 1)
-      (outputdirectory "")
+      (outputdirectory "Manufacturing/")
     )
   )
@@
     (descr "Capacitor SMD 0805 (2012 Metric), square (rectangular) end terminal, IPC_7351 nominal, (Body size source: IPC-SM-782 page 76, https://www.pcb-3d.com/wordpress/wp-content/uploads/ipc-sm-782a_amendment_1_and_2.pdf, https://docs.google.com/spreadsheets/d/1BsfQQcO9C6DZCsRaXUlFlo91Tg2WpOkGARC1WS5S8t0/edit?usp=sharing), generated with kicad-footprint-generator")
     (tags "capacitor")
+    (property "LCSC" "C1711")
     (property "Sheetfile" "CAN.kicad_sch")
     (property "Sheetname" "CAN")
@@
     (descr "JST PH series connector, B5B-PH-K (http://www.jst-mfg.com/product/pdf/eng/ePH.pdf), generated with kicad-footprint-generator")
     (tags "connector JST PH side entry")
+    (property "LCSC" "C157993")
     (property "Sheetfile" "CAN.kicad_sch")
     (property "Sheetname" "CAN")
@@
     (fp_line (start 9.95 2.8) (end 9.95 -1.7)
       (stroke (width 0.1) (type solid)) (layer "F.Fab"))
-    (pad "1" thru_hole roundrect (at 0 0 270) (size 1.2 1.75) (drill 0.75) (layers "*.Cu" "*.Mask") (roundrect_rratio 0.208333)
+    (pad "1" thru_hole roundrect (at 0 0 270) (size 1.2 1.75) (drill 0.75) (layers "*.Cu" "*.Mask") (roundrect_rratio 0.2083333333)
       (net 6 "+12V") (pinfunction "Pin_1") (pintype "passive"))
     (pad "2" thru_hole oval (at 2 0 270) (size 1.2 1.75) (drill 0.75) (layers "*.Cu" "*.Mask")
@@
     (at 141.775 90.1875)
     (descr "aka SOT782-1")
+    (property "LCSC" "C3229259")
     (property "Sheetfile" "CAN.kicad_sch")
     (property "Sheetname" "CAN")
@@
     (descr "SOT, 3 Pin (https://www.jedec.org/system/files/docs/to-236h.pdf variant AB), generated with kicad-footprint-generator ipc_gullwing_generator.py")
     (tags "SOT TO_SOT_SMD")
+    (property "LCSC" "C552486")
     (property "Sheetfile" "CAN.kicad_sch")
     (property "Sheetname" "CAN")
@@
     (descr "Resistor SMD 0805 (2012 Metric), square (rectangular) end terminal, IPC_7351 nominal, (Body size source: IPC-SM-782 page 72, https://www.pcb-3d.com/wordpress/wp-content/uploads/ipc-sm-782a_amendment_1_and_2.pdf), generated with kicad-footprint-generator")
     (tags "resistor")
+    (property "LCSC" "C17414")
     (property "Sheetfile" "CAN.kicad_sch")
     (property "Sheetname" "CAN")
@@
     (fp_line (start 1 0.625) (end -1 0.625)
       (stroke (width 0.1) (type solid)) (layer "F.Fab"))
-    (pad "1" smd roundrect (at -0.9125 0 90) (size 1.025 1.4) (layers "F.Cu" "F.Paste" "F.Mask") (roundrect_rratio 0.243902)
+    (pad "1" smd roundrect (at -0.9125 0 90) (size 1.025 1.4) (layers "F.Cu" "F.Paste" "F.Mask") (roundrect_rratio 0.243902439)
       (net 2 "GND") (pintype "passive"))
-    (pad "2" smd roundrect (at 0.9125 0 90) (size 1.025 1.4) (layers "F.Cu" "F.Paste" "F.Mask") (roundrect_rratio 0.243902)
+    (pad "2" smd roundrect (at 0.9125 0 90) (size 1.025 1.4) (layers "F.Cu" "F.Paste" "F.Mask") (roundrect_rratio 0.243902439)
       (net 10 "Net-(U3-STB)") (pintype "passive"))
     (model "${KICAD6_3DMODEL_DIR}/Resistor_SMD.3dshapes/R_0805_2012Metric.wrl"
@@
     (descr "JST PH series connector, B5B-PH-K (http://www.jst-mfg.com/product/pdf/eng/ePH.pdf), generated with kicad-footprint-generator")
     (tags "connector JST PH side entry")
+    (property "LCSC" "C157993")
     (property "Sheetfile" "CAN.kicad_sch")
     (property "Sheetname" "CAN")
@@
     (fp_line (start 9.95 2.8) (end 9.95 -1.7)
       (stroke (width 0.1) (type solid)) (layer "F.Fab"))
-    (pad "1" thru_hole roundrect (at 0 0 270) (size 1.2 1.75) (drill 0.75) (layers "*.Cu" "*.Mask") (roundrect_rratio 0.208333)
+    (pad "1" thru_hole roundrect (at 0 0 270) (size 1.2 1.75) (drill 0.75) (layers "*.Cu" "*.Mask") (roundrect_rratio 0.2083333333)
       (net 6 "+12V") (pinfunction "Pin_1") (pintype "passive"))
     (pad "2" thru_hole oval (at 2 0 270) (size 1.2 1.75) (drill 0.75) (layers "*.Cu" "*.Mask")
@@
     (descr "Capacitor SMD 0805 (2012 Metric), square (rectangular) end terminal, IPC_7351 nominal, (Body size source: IPC-SM-782 page 76, https://www.pcb-3d.com/wordpress/wp-content/uploads/ipc-sm-782a_amendment_1_and_2.pdf, https://docs.google.com/spreadsheets/d/1BsfQQcO9C6DZCsRaXUlFlo91Tg2WpOkGARC1WS5S8t0/edit?usp=sharing), generated with kicad-footprint-generator")
     (tags "capacitor")
+    (property "LCSC" "C1711")
     (property "Sheetfile" "CAN.kicad_sch")
     (property "Sheetname" "CAN")
@@
     (descr "Resistor SMD 0805 (2012 Metric), square (rectangular) end terminal, IPC_7351 nominal, (Body size source: IPC-SM-782 page 72, https://www.pcb-3d.com/wordpress/wp-content/uploads/ipc-sm-782a_amendment_1_and_2.pdf), generated with kicad-footprint-generator")
     (tags "resistor")
+    (property "LCSC" "C17437")
     (property "Sheetfile" "CAN.kicad_sch")
     (property "Sheetname" "CAN")
@@
     (fp_line (start 1 0.625) (end -1 0.625)
       (stroke (width 0.1) (type solid)) (layer "F.Fab"))
-    (pad "1" smd roundrect (at -0.9125 0) (size 1.025 1.4) (layers "F.Cu" "F.Paste" "F.Mask") (roundrect_rratio 0.243902)
+    (pad "1" smd roundrect (at -0.9125 0) (size 1.025 1.4) (layers "F.Cu" "F.Paste" "F.Mask") (roundrect_rratio 0.243902439)
       (net 7 "/CAN/CAN_L") (pintype "passive"))
-    (pad "2" smd roundrect (at 0.9125 0) (size 1.025 1.4) (layers "F.Cu" "F.Paste" "F.Mask") (roundrect_rratio 0.243902)
+    (pad "2" smd roundrect (at 0.9125 0) (size 1.025 1.4) (layers "F.Cu" "F.Paste" "F.Mask") (roundrect_rratio 0.243902439)
       (net 4 "Net-(J2-Pin_1)") (pintype "passive"))
     (model "${KICAD6_3DMODEL_DIR}/Resistor_SMD.3dshapes/R_0805_2012Metric.wrl"
@@
     (at 140.2597 84.02375 90)
     (descr "CAN and CANFD Common Mode Choke")
+    (property "LCSC" "C95572")
     (property "Sheetfile" "CAN.kicad_sch")
     (property "Sheetname" "CAN")

Commit message: Added fiducials to all boards.
Parts:
- added FID1: Fiducial, Fiducial:Fiducial_0.5mm_Mask1mm, F.Cu at (118.4, 70.4)
- added FID2: Fiducial, Fiducial:Fiducial_0.5mm_Mask1mm, F.Cu at (150.6, 70.4)
- added FID3: Fiducial, Fiducial:Fiducial_0.5mm_Mask1mm, F.Cu at (111.4, 117.8)
Changed lines of the file:
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@@
   (footprint "Britishideas:Teensy_4.0" (layer "F.Cu")
     (at 116.42 84.73)
+    (property "LCSC" "")
     (property "Sheetfile" "IMU.kicad_sch")
     (property "Sheetname" "")
@@
     (descr "Through hole straight pin header, 1x02, 2.54mm pitch, single row")
     (tags "Through hole pin header THT 1x02 2.54mm single row")
+    (property "LCSC" "C7494857")
     (property "Sheetfile" "IMU.kicad_sch")
     (property "Sheetname" "")
@@
     )
   )
+  (footprint "Fiducial:Fiducial_0.5mm_Mask1mm" (layer "F.Cu")
+    (at 111.4 117.8)
+    (descr "Circular Fiducial, 0.5mm bare copper, 1mm soldermask opening (Level C)")
+    (tags "fiducial")
+    (property "Sheetfile" "IMU.kicad_sch")
+    (property "Sheetname" "")
+    (property "ki_description" "Fiducial Marker")
+    (property "ki_keywords" "fiducial marker")
+    (attr smd)
+    (fp_text reference "FID3" (at 0 -1.5) (layer "F.SilkS") hide
+        (effects (font (size 1 1) (thickness 0.15)))
+    )
+    (fp_text value "Fiducial" (at 0 1.5) (layer "F.Fab")
+        (effects (font (size 1 1) (thickness 0.15)))
+    )
+    (fp_text user "${REFERENCE}" (at 0 0) (layer "F.Fab")
+        (effects (font (size 0.2 0.2) (thickness 0.04)))
+    )
+    (fp_circle (center 0 0) (end 0.75 0)
+      (stroke (width 0.05) (type solid)) (fill none) (layer "F.CrtYd"))
+    (fp_circle (center 0 0) (end 0.5 0)
+      (stroke (width 0.1) (type solid)) (fill none) (layer "F.Fab"))
+    (pad "" smd circle (at 0 0) (size 0.5 0.5) (layers "F.Cu" "F.Mask")
+      (solder_mask_margin 0.25) (clearance 0.25))
+  )
   (footprint "Resistor_SMD:R_0805_2012Metric" (layer "F.Cu")
     (at 140 88.75 90)
@@
     (property "ki_description" "Resistor")
     (property "ki_keywords" "R res resistor")
+    (property "manf#" "")
     (attr smd)
     (fp_text reference "R1" (at 0 -1.65 90) (layer "F.SilkS")
@@
     (descr "Through hole straight pin header, 1x02, 2.54mm pitch, single row")
     (tags "Through hole pin header THT 1x02 2.54mm single row")
+    (property "LCSC" "C7494857")
     (property "Sheetfile" "CAN.kicad_sch")
     (property "Sheetname" "CAN")
@@
   (footprint "Britishideas:Adafruit_BNO085" (layer "F.Cu")
     (at 155.5 112.7 180)
+    (property "LCSC" "")
     (property "Sheetfile" "IMU.kicad_sch")
     (property "Sheetname" "")
@@
     )
   )
+  (footprint "Fiducial:Fiducial_0.5mm_Mask1mm" (layer "F.Cu")
+    (at 150.6 70.4)
+    (descr "Circular Fiducial, 0.5mm bare copper, 1mm soldermask opening (Level C)")
+    (tags "fiducial")
+    (property "Sheetfile" "IMU.kicad_sch")
+    (property "Sheetname" "")
+    (property "ki_description" "Fiducial Marker")
+    (property "ki_keywords" "fiducial marker")
+    (attr smd)
+    (fp_text reference "FID2" (at 0 -1.5) (layer "F.SilkS") hide
+        (effects (font (size 1 1) (thickness 0.15)))
+    )
+    (fp_text value "Fiducial" (at 0 1.5) (layer "F.Fab")
+        (effects (font (size 1 1) (thickness 0.15)))
+    )
+    (fp_text user "${REFERENCE}" (at 0 0) (layer "F.Fab")
+        (effects (font (size 0.2 0.2) (thickness 0.04)))
+    )
+    (fp_circle (center 0 0) (end 0.75 0)
+      (stroke (width 0.05) (type solid)) (fill none) (layer "F.CrtYd"))
+    (fp_circle (center 0 0) (end 0.5 0)
+      (stroke (width 0.1) (type solid)) (fill none) (layer "F.Fab"))
+    (pad "" smd circle (at 0 0) (size 0.5 0.5) (layers "F.Cu" "F.Mask")
+      (solder_mask_margin 0.25) (clearance 0.25))
+  )
   (footprint "EmSA:ACT1210-510-2P-TL00" (layer "F.Cu")
     (at 140.2597 84.02375 90)
@@
     )
   )
+  (footprint "Fiducial:Fiducial_0.5mm_Mask1mm" (layer "F.Cu")
+    (at 118.4 70.4)
+    (descr "Circular Fiducial, 0.5mm bare copper, 1mm soldermask opening (Level C)")
+    (tags "fiducial")
+    (property "Sheetfile" "IMU.kicad_sch")
+    (property "Sheetname" "")
+    (property "ki_description" "Fiducial Marker")
+    (property "ki_keywords" "fiducial marker")
+    (attr smd)
+    (fp_text reference "FID1" (at 0 -1.5) (layer "F.SilkS") hide
+        (effects (font (size 1 1) (thickness 0.15)))
+    )
+    (fp_text value "Fiducial" (at 0 1.5) (layer "F.Fab")
+        (effects (font (size 1 1) (thickness 0.15)))
+    )
+    (fp_text user "${REFERENCE}" (at 0 0) (layer "F.Fab")
+        (effects (font (size 0.2 0.2) (thickness 0.04)))
+    )
+    (fp_circle (center 0 0) (end 0.75 0)
+      (stroke (width 0.05) (type solid)) (fill none) (layer "F.CrtYd"))
+    (fp_circle (center 0 0) (end 0.5 0)
+      (stroke (width 0.1) (type solid)) (fill none) (layer "F.Fab"))
+    (pad "" smd circle (at 0 0) (size 0.5 0.5) (layers "F.Cu" "F.Mask")
+      (solder_mask_margin 0.25) (clearance 0.25))
+  )
   (gr_line (start 112.25 90.25) (end 110.75 94.25)
