File: Electronics/User Controls/CAN.kicad_sch (KiCad schematic)
At the start: 9 parts, among them J1 TERM, J2 CAN BUS, U1 TJA1462ATK-0Z, U2 PESD2CANFD24V-TR

Commit message: Added 4.7uF caps to FT232RL on controller.
Parts:
- C1, C2: LCSC (none) -> C1711
- J1: LCSC (none) -> C7494857
- J2: LCSC (none) -> C157993
- L1: LCSC (none) -> C95572
- R1: LCSC (none) -> C17414
- R2: LCSC (none) -> C17437
- U1: LCSC (none) -> C3229259
- U2: LCSC (none) -> C552486
Changed lines of the file:
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@@
+      (effects (font (size 1.27 1.27)) hide)
+    )
+    (property "LCSC" "C95572" (at 130.81 90.17 0)
       (effects (font (size 1.27 1.27)) hide)
     )
@@
       (effects (font (size 1.27 1.27)) hide)
     )
+    (property "LCSC" "C17437" (at 185.42 81.28 0)
+      (effects (font (size 1.27 1.27)) hide)
+    )
     (pin "1")
     (pin "2")
@@
     )
     (property "Datasheet" "~" (at 91.44 128.905 0)
+      (effects (font (size 1.27 1.27)) hide)
+    )
+    (property "LCSC" "C1711" (at 91.44 128.905 0)
       (effects (font (size 1.27 1.27)) hide)
     )
@@
       (effects (font (size 1.27 1.27)) hide)
     )
+    (property "LCSC" "C17414" (at 109.22 99.06 0)
+      (effects (font (size 1.27 1.27)) hide)
+    )
     (pin "1")
     (pin "2")
@@
     )
     (property "Datasheet" "~" (at 185.42 71.12 0)
+      (effects (font (size 1.27 1.27)) hide)
+    )
+    (property "LCSC" "C7494857" (at 185.42 71.12 0)
       (effects (font (size 1.27 1.27)) hide)
     )
@@
       (effects (font (size 1.27 1.27)) hide)
     )
+    (property "LCSC" "C157993" (at 240.665 87.63 0)
+      (effects (font (size 1.27 1.27)) hide)
+    )
     (pin "2")
     (pin "5")
@@
       (effects (font (size 1.27 1.27)) hide)
     )
+    (property "LCSC" "C1711" (at 80.645 128.905 0)
+      (effects (font (size 1.27 1.27)) hide)
+    )
     (pin "1")
     (pin "2")
@@
     )
     (property "manf#" "TJA1462ATK/0Z" (at 87.63 80.01 0)
+      (effects (font (size 1.27 1.27)) hide)
+    )
+    (property "LCSC" "C3229259" (at 80.01 95.25 0)
       (effects (font (size 1.27 1.27)) hide)
     )
@@
       (effects (font (size 1.27 1.27)) hide)
     )
+    (property "LCSC" "C552486" (at 150.495 102.87 0)
+      (effects (font (size 1.27 1.27)) hide)
+    )
