File: Electronics/User Controls/User Controls.kicad_sch (KiCad schematic)
At the start: 20 parts, among them J10 BUTTON 7, J11 BUTTON 8, J12 JOYSTICK 1, J13 JOYSTICK 2, J3 Conn_01x02, J4 BUTTON 1, J5 BUTTON 2, J6 BUTTON 3, J7 BUTTON 4, J8 BUTTON 5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

Commit message: Added 4.7uF caps to FT232RL on controller.
Parts:
- J10, J11, J4, J5, J6, J7, J8, J9: LCSC (none) -> C131334
- J12, J13: LCSC (none) -> C157993
- J3: LCSC (none) -> C7494857
- R10, R3, R4, R5, R6, R7, R8, R9: LCSC (none) -> C17414
- U3: LCSC (none) -> C2897377
Changed lines of the file:
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@@
+      (effects (font (size 1.27 1.27)) hide)
+    )
+    (property "LCSC" "C17414" (at 51.435 41.275 0)
       (effects (font (size 1.27 1.27)) hide)
     )
@@
     )
     (property "manf#" "B5B-PH-K-S" (at 125.73 127 0)
+      (effects (font (size 1.27 1.27)) hide)
+    )
+    (property "LCSC" "C157993" (at 125.73 127 0)
       (effects (font (size 1.27 1.27)) hide)
     )
@@
       (effects (font (size 1.27 1.27)) hide)
     )
+    (property "LCSC" "C17414" (at 92.71 116.205 0)
+      (effects (font (size 1.27 1.27)) hide)
+    )
     (pin "1")
     (pin "2")
@@
       (effects (font (size 1.27 1.27)) hide)
     )
+    (property "LCSC" "C17414" (at 92.71 153.67 0)
+      (effects (font (size 1.27 1.27)) hide)
+    )
     (pin "1")
     (pin "2")
@@
       (effects (font (size 1.27 1.27)) hide)
     )
+    (property "LCSC" "C17414" (at 51.435 78.105 0)
+      (effects (font (size 1.27 1.27)) hide)
+    )
     (pin "1")
     (pin "2")
@@
     )
     (property "manf#" "B4B-PH-K-S" (at 76.2 125.73 0)
+      (effects (font (size 1.27 1.27)) hide)
+    )
+    (property "LCSC" "C131334" (at 76.2 125.73 0)
       (effects (font (size 1.27 1.27)) hide)
     )
@@
       (effects (font (size 1.27 1.27)) hide)
     )
+    (property "LCSC" "C17414" (at 51.435 116.205 0)
+      (effects (font (size 1.27 1.27)) hide)
+    )
     (pin "1")
     (pin "2")
@@
       (effects (font (size 1.27 1.27)) hide)
     )
+    (property "LCSC" "C17414" (at 92.71 41.275 0)
+      (effects (font (size 1.27 1.27)) hide)
+    )
     (pin "1")
     (pin "2")
@@
       (effects (font (size 1.27 1.27)) hide)
     )
+    (property "LCSC" "C17414" (at 92.71 78.105 0)
+      (effects (font (size 1.27 1.27)) hide)
+    )
     (pin "1")
     (pin "2")
@@
     )
     (property "Datasheet" "" (at 160.655 179.07 0)
+      (effects (font (size 1.27 1.27)) hide)
+    )
+    (property "LCSC" "C2897377" (at 160.655 179.07 0)
       (effects (font (size 1.27 1.27)) hide)
     )
@@
       (effects (font (size 1.27 1.27)) hide)
     )
+    (property "LCSC" "C157993" (at 125.73 164.465 0)
+      (effects (font (size 1.27 1.27)) hide)
+    )
     (pin "2")
     (pin "5")
@@
       (effects (font (size 1.27 1.27)) hide)
     )
+    (property "LCSC" "C131334" (at 34.925 125.73 0)
+      (effects (font (size 1.27 1.27)) hide)
+    )
     (pin "2")
     (pin "3")
@@
       (effects (font (size 1.27 1.27)) hide)
     )
+    (property "LCSC" "C7494857" (at 175.895 48.895 0)
+      (effects (font (size 1.27 1.27)) hide)
+    )
     (pin "1")
     (pin "2")
@@
     )
     (property "manf#" "B4B-PH-K-S" (at 76.2 163.195 0)
+      (effects (font (size 1.27 1.27)) hide)
+    )
+    (property "LCSC" "C131334" (at 76.2 163.195 0)
       (effects (font (size 1.27 1.27)) hide)
     )
@@
       (effects (font (size 1.27 1.27)) hide)
     )
+    (property "LCSC" "C131334" (at 34.925 163.195 0)
+      (effects (font (size 1.27 1.27)) hide)
+    )
     (pin "2")
     (pin "3")
@@
       (effects (font (size 1.27 1.27)) hide)
     )
+    (property "LCSC" "C17414" (at 51.435 153.67 0)
+      (effects (font (size 1.27 1.27)) hide)
+    )
     (pin "1")
     (pin "2")
@@
     )
     (property "manf#" "B4B-PH-K-S" (at 76.2 50.8 0)
+      (effects (font (size 1.27 1.27)) hide)
+    )
+    (property "LCSC" "C131334" (at 76.2 50.8 0)
       (effects (font (size 1.27 1.27)) hide)
     )
@@
       (effects (font (size 1.27 1.27)) hide)
     )
+    (property "LCSC" "C131334" (at 34.925 50.8 0)
+      (effects (font (size 1.27 1.27)) hide)
+    )
     (pin "2")
     (pin "3")
@@
       (effects (font (size 1.27 1.27)) hide)
     )
+    (property "LCSC" "C131334" (at 34.925 87.63 0)
+      (effects (font (size 1.27 1.27)) hide)
+    )
     (pin "2")
     (pin "3")
@@
       (effects (font (size 1.27 1.27)) hide)
     )
+    (property "LCSC" "C131334" (at 76.2 87.63 0)
+      (effects (font (size 1.27 1.27)) hide)
+    )

Commit message: Removed JLCPCB part numbers for Teensy and BNO085 connectors. Added JLCPCB part number for 4.7uF capacitor. Generated JLCPCB manufacturing files for all boards.
Parts:
- U3: LCSC C2897377 -> (none)
Changed lines of the file:
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@@
       (effects (font (size 1.27 1.27)) hide)
     )
-    (property "LCSC" "C2897377" (at 160.655 179.07 0)
+    (property "LCSC" "" (at 160.655 179.07 0)
       (effects (font (size 1.27 1.27)) hide)
     )

Commit message: Added fiducials to all boards.
Parts:
- added FID1, FID2, FID3: Fiducial, Fiducial:Fiducial_0.5mm_Mask1mm, symbol Mechanical:Fiducial
Changed lines of the file:
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@@
   (title_block
     (title "Tandem Leveller User Controls")
-    (date "2025-02-25")
+    (date "2025-03-13")
     (rev "V1.0")
     (company "(C) andy@britishideas.com 2025")
@@
     )
   )
+  (symbol (lib_id "Mechanical:Fiducial") (at 160.655 188.595 0) (unit 1)
+    (in_bom yes) (on_board yes) (dnp no) (fields_autoplaced)
+    (property "Reference" "FID3" (at 163.195 187.325 0)
+      (effects (font (size 1.27 1.27)) (justify left))
+    )
+    (property "Value" "Fiducial" (at 163.195 189.865 0)
+      (effects (font (size 1.27 1.27)) (justify left))
+    )
+    (property "Footprint" "Fiducial:Fiducial_0.5mm_Mask1mm" (at 160.655 188.595 0)
+      (effects (font (size 1.27 1.27)) hide)
+    )
+    (property "Datasheet" "~" (at 160.655 188.595 0)
+      (effects (font (size 1.27 1.27)) hide)
+    )
+    (instances
+      (project "User Controls"
+        (path "/6eedea76-9308-4a57-b0c3-a2def9dafc46"
+          (reference "FID3") (unit 1)
+        )
+      )
+    )
+  )
   (symbol (lib_id "power:+5V") (at 140.97 119.38 0) (unit 1)
     (in_bom yes) (on_board yes) (dnp no)
@@
     )
   )
+  (symbol (lib_id "Mechanical:Fiducial") (at 136.525 188.595 0) (unit 1)
+    (in_bom yes) (on_board yes) (dnp no) (fields_autoplaced)
+    (property "Reference" "FID1" (at 139.065 187.325 0)
+      (effects (font (size 1.27 1.27)) (justify left))
+    )
+    (property "Value" "Fiducial" (at 139.065 189.865 0)
+      (effects (font (size 1.27 1.27)) (justify left))
+    )
+    (property "Footprint" "Fiducial:Fiducial_0.5mm_Mask1mm" (at 136.525 188.595 0)
+      (effects (font (size 1.27 1.27)) hide)
+    )
+    (property "Datasheet" "~" (at 136.525 188.595 0)
+      (effects (font (size 1.27 1.27)) hide)
+    )
+    (instances
+      (project "User Controls"
+        (path "/6eedea76-9308-4a57-b0c3-a2def9dafc46"
+          (reference "FID1") (unit 1)
+        )
+      )
+    )
+  )
   (symbol (lib_id "power:GND") (at 99.06 170.18 0) (unit 1)
     (in_bom yes) (on_board yes) (dnp no)
@@
         )
       )
+    )
+  )
+  (symbol (lib_id "Mechanical:Fiducial") (at 148.59 188.595 0) (unit 1)
+    (in_bom yes) (on_board yes) (dnp no) (fields_autoplaced)
+    (property "Reference" "FID2" (at 151.13 187.325 0)
+      (effects (font (size 1.27 1.27)) (justify left))
+    )
+    (property "Value" "Fiducial" (at 151.13 189.865 0)
+      (effects (font (size 1.27 1.27)) (justify left))
+    )
+    (property "Footprint" "Fiducial:Fiducial_0.5mm_Mask1mm" (at 148.59 188.595 0)
+      (effects (font (size 1.27 1.27)) hide)
+    )
+    (property "Datasheet" "~" (at 148.59 188.595 0)
+      (effects (font (size 1.27 1.27)) hide)
+    )
+    (instances
+      (project "User Controls"
+        (path "/6eedea76-9308-4a57-b0c3-a2def9dafc46"
+          (reference "FID2") (unit 1)
+        )
+      )
