File: Electronics/Scraper Angle/Scraper Angle.kicad_sch (KiCad schematic)
At the start: 10 parts, among them J12 SENSOR, J3 Conn_01x02, J4 Conn_01x02, J5 Conn_01x02, U3 TEENSY 4.0

Commit message: Changed sensor connector on scraper angle board. Generated production files for scraper angle board.
Parts:
- J12: footprint Connector_JST:JST_EH_B3B-EH-A_1x03_P2.50mm_Vertical -> Connector_JST:JST_PH_B3B-PH-K_1x03_P2.00mm_Vertical; LCSC (none) -> C131339
Changed lines of the file:
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@@
   (title_block
     (title "Tandem Leveller Scraper Angle")
-    (date "2025-10-14")
+    (date "2025-10-20")
     (rev "V1.0")
     (company "(C) andy@britishideas.com 2025")
@@
       (effects (font (size 1.27 1.27)) (justify left))
     )
-    (property "Footprint" "Connector_JST:JST_EH_B3B-EH-A_1x03_P2.50mm_Vertical" (at 216.535 119.38 0)
+    (property "Footprint" "Connector_JST:JST_PH_B3B-PH-K_1x03_P2.00mm_Vertical" (at 216.535 119.38 0)
       (effects (font (size 1.27 1.27)) hide)
     )
@@
       (effects (font (size 1.27 1.27)) hide)
     )
-    (property "LCSC" "" (at 216.535 119.38 0)
+    (property "LCSC" "C131339" (at 216.535 119.38 0)
       (effects (font (size 1.27 1.27)) hide)
     )
