File: Electronics/Controller V2/GNSS Daughterboard/GNSS Daughterboard.kicad_sch (KiCad schematic)
At the start: 13 parts, among them J1 GNSS, J2 Conn_01x02, J3 Conn_01x02, J4 Conn_01x02, J5 Conn_01x02, J6 Conn_01x02, J7 Conn_01x02, J8 GNSS, U1 simpleRTK2B

Commit message: Completed daughterboards.
Parts:
- H1, H2, H3, H4: footprint MountingHole:MountingHole_3.2mm_M3 -> MountingHole:MountingHole_6.4mm_M6
Changed lines of the file:
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@@
       (effects (font (size 1.27 1.27)) (justify left))
     )
-    (property "Footprint" "MountingHole:MountingHole_3.2mm_M3" (at 144.145 131.445 0)
+    (property "Footprint" "MountingHole:MountingHole_6.4mm_M6" (at 144.145 131.445 0)
       (effects (font (size 1.27 1.27)) hide)
     )
@@
       (effects (font (size 1.27 1.27)) (justify left))
     )
-    (property "Footprint" "MountingHole:MountingHole_3.2mm_M3" (at 165.1 131.445 0)
+    (property "Footprint" "MountingHole:MountingHole_6.4mm_M6" (at 165.1 131.445 0)
       (effects (font (size 1.27 1.27)) hide)
     )
@@
       (effects (font (size 1.27 1.27)) (justify left))
     )
-    (property "Footprint" "MountingHole:MountingHole_3.2mm_M3" (at 144.145 137.795 0)
+    (property "Footprint" "MountingHole:MountingHole_6.4mm_M6" (at 144.145 137.795 0)
       (effects (font (size 1.27 1.27)) hide)
     )
@@
       (effects (font (size 1.27 1.27)) (justify left))
     )
-    (property "Footprint" "MountingHole:MountingHole_3.2mm_M3" (at 165.1 137.795 0)
-      (effects (font (size 1.27 1.27)) hide)
-    )
+    (property "Footprint" "MountingHole:MountingHole_6.4mm_M6" (at 165.1 137.795 0)
+      (effects (font (size 1.27 1.27)) hide)
+    )
