File: Electronics/Controller V2/Motherboard/Tandem Leveller Controller V2.kicad_pcb (KiCad board)
At the start: 6 copper layers, 230.5 x 129 mm, 96 parts, among them J1 Conn_01x08, J10 ORIENT, J11 OPT, J12 IMU, J14 TABLET 1 PWR, J15 TABLET 2 PWR, J2 Conn_01x10, J3 GNSS, J4 TERM, J5 Pulse_J0011D01BNL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

Commit message: Added current sensing for valve E.
Parts:
- added C16: 100n, Capacitor_SMD:C_0805_2012Metric, F.Cu at (236.0, 77.8)
- added C17: 1n, Capacitor_SMD:C_0805_2012Metric, F.Cu at (236.0, 83.0)
- added U12: ACS712xLCTR-20A, Package_SO:SOIC-8_3.9x4.9mm_P1.27mm, F.Cu at (231.0, 81.0)
Connections:
- J2 pad 9: /VALVE_E_MB -> /Valves/VALVE_E_MB
- J9 pad 7: /VALVE_E_MB -> /VALVE_E_MB_OUT
- U11 pad 6: unconnected-(U11-AIN2-Pad6) -> Net-(U11-AIN2)
Routing:
- net /VALVE_E_MB: track 107.2 -> 0.00 mm
- net /VALVE_E_MB_OUT: track 0.00 -> 92.9 mm, vias 0 -> 1
- net Net-(U11-AIN2): track 0.00 -> 61.0 mm, vias 0 -> 2
- net /Valves/VALVE_E_MB: track 0.00 -> 23.5 mm, vias 0 -> 1
- net +5V: track 25.6 -> 29.5 mm, vias 13 -> 14
- net Net-(U12-FILTER): track 0.00 -> 2.70 mm
- net GND: vias 253 -> 261
