File: Electronics/Controller V2/Motherboard/GNSS.kicad_sch (KiCad schematic)
At the start: 6 parts, among them J3 GNSS, U2 simpleRTK2B

Commit message: Added generic IMU option.
Connections:
- net GPIO_G1 renamed GPIO_G1_RX
- net GPIO_G2 renamed GPIO_G2_TX
Changed lines of the file:
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@@
   (title_block
     (title "Tandem Leveller Controller")
-    (date "2026-02-06")
+    (date "2026-02-09")
     (rev "V2.0")
     (company "(C) andy@britishideas.com 2026")
@@
     (effects (font (size 1.27 1.27)) (justify right))
   )
-  (hierarchical_label "GPIO_G2" (shape bidirectional) (at 125.095 102.87 0) (fields_autoplaced)
+  (hierarchical_label "GPIO_G2_TX" (shape bidirectional) (at 125.095 102.87 0) (fields_autoplaced)
     (effects (font (size 1.27 1.27)) (justify left))
   )
@@
     (effects (font (size 1.27 1.27)) (justify left))
   )
-  (hierarchical_label "GPIO_G1" (shape bidirectional) (at 125.095 100.33 0) (fields_autoplaced)
+  (hierarchical_label "GPIO_G1_RX" (shape bidirectional) (at 125.095 100.33 0) (fields_autoplaced)
     (effects (font (size 1.27 1.27)) (justify left))
   )
